Commit message: verified bot motion with rviz

File: src/jetPR_description/urdf/jetPR.urdf (robot description, URDF)
Before this commit: robot pepper, 3 links, 2 joints
Links:
- link base_link: geometry visual mesh filename=package://jetPR_description/meshes/chassisv2.STL scale=0.001 0.001 0.001
- link left_wheel: geometry visual mesh filename=package://jetPR_description/meshes/wheel.STL scale=0.001 0.001 0.001
- link right_wheel: geometry visual mesh filename=package://jetPR_description/meshes/wheel.STL scale=0.001 0.001 0.001

Commit message: modified urdf to add camera base link

File: src/jetPR_description/urdf/jetPR.urdf (robot description, URDF)
Before this commit: robot jetPR, 3 links, 2 joints
Links:
- added link camera_base_link
Joints:
- added joint camera_base_joint: type continuous, parent base_link, child camera_base_link, origin xyz=0.035 0 0.285 rpy=0 0 0, axis 0.0 1.0 0

Commit message: modified urdf

File: src/jetPR_description/urdf/jetPR.urdf (robot description, URDF)
Before this commit: robot jetPR, 4 links, 3 joints
Links:
- removed link camera_base_link
- added link camera_link
Joints:
- joint camera_base_joint: child camera_base_link -> camera_link

Commit message: added caster and gazebo interface

File: src/jetPR_description/urdf/jetPR.urdf (robot description, URDF)
Before this commit: robot jetPR, 4 links, 3 joints
Links:
- removed link camera_link
- added link camera_base_link
- link base_link: mass None -> 5; geometry collision mesh filename=package://jetPR_description/meshes/chassisv2.STL scale=0.001 0.001 0.001; collision sphere radius=0.005
- link left_wheel: mass None -> 0.3; geometry collision mesh filename=package://jetPR_description/meshes/wheel.STL scale=0.001 0.001 0.001; visual mesh filename=package://jetPR_description/meshes/wheel.STL scale=0.001 0.001 0.001
- link right_wheel: mass None -> 0.3; geometry collision mesh filename=package://jetPR_description/meshes/wheel.STL scale=0.001 0.001 0.001; visual mesh filename=package://jetPR_description/meshes/wheel.STL scale=0.001 0.001 0.001
Joints:
- joint camera_base_joint: child camera_link -> camera_base_link
